File: src/temperature/kicad/rf_temperature.kicad_sch (KiCad schematic)
At the start: 13 parts, among them J1 Conn_01x20, J2 Conn_01x20, J2 Screw_Terminal_01x02, U1 Pico, U2 DS18B20, U3 NRF24L01_Breakout

Commit message: use ground plane
Parts:
- U4: footprint MyLibrary:LM2596AdjBuck -> my_LM2596_Library:my_LM2596AdjBuck; symbol my_library:LM2596AdjBuck -> my_LM2596:LM2596AdjBuck
Changed lines of the file:
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@@
   (title_block
     (title "RF Temp")
-    (date "2023-02-26")
-    (rev "0.3")
+    (date "2023-03-25")
+    (rev "0.4")
   )
   (junction (at 137.16 140.97) (diameter 0) (color 0 0 0 0)
@@
     )
   )
-  (symbol (lib_id "my_library:LM2596AdjBuck") (at 124.46 20.32 0) (unit 1)
+  (symbol (lib_id "my_LM2596:LM2596AdjBuck") (at 124.46 20.32 0) (unit 1)
     (in_bom yes) (on_board yes) (dnp no) (fields_autoplaced)
-    (property "Reference" "U4" (at 123.19 21.59 0)
+    (property "Reference" "U4" (at 124.46 20.32 0)
       (effects (font (size 1.27 1.27)))
     )
@@
       (effects (font (size 1.27 1.27)))
     )
-    (property "Footprint" "MyLibrary:LM2596AdjBuck" (at 124.46 20.32 0)
-      (effects (font (size 1.27 1.27)) hide)
-    )
+    (property "Footprint" "my_LM2596_Library:my_LM2596AdjBuck" (at 124.46 20.32 0)
+      (effects (font (size 1.27 1.27)) hide)
+    )
